Commit message: UR5e+Robotiq夹爪集成：更新URDF模型、MoveIt配置和Gazebo启动文件

File: src/arm_urdf/urdf/arm.urdf (robot description, URDF)
Before this commit: robot episode_urdf_0523, 8 links, 7 joints
Links:
- added link gripper_left, mass 0.01; collision box size=0.01 0.005 0.08; visual box size=0.01 0.005 0.08
- added link gripper_right, mass 0.01; collision box size=0.01 0.005 0.08; visual box size=0.01 0.005 0.08
Joints:
- added joint gripper_left_joint: type prismatic, parent L6, child gripper_left, origin xyz=0.0 0.05 0.0 rpy=0 0 0, axis 0 -1 0, limit lower=0 upper=0.0475 effort=50 velocity=0.05
- added joint gripper_right_joint: type prismatic, parent L6, child gripper_right, origin xyz=0.0 -0.05 0.0 rpy=0 0 0, axis 0 1 0, limit lower=0 upper=0.0475 effort=50 velocity=0.05

File: src/my_robot_moveit_config/config/episode_urdf_0523.ros2_control.xacro (robot description, xacro)
@@ -1,9 +1,19 @@
 <?xml version="1.0"?>
 <robot xmlns:xacro="http://www.ros.org/wiki/xacro">
-    <xacro:macro name="episode_urdf_0523_ros2_control" params="name initial_positions_file">
+    <xacro:macro name="episode_urdf_0523_ros2_control" params="name initial_positions_file sim_backend:=gazebo">
         <xacro:property name="initial_positions" value="${xacro.load_yaml(initial_positions_file)['initial_positions']}"/>
+        <!-- 根据 sim_backend 选择硬件插件: gazebo → GazeboSystem, mock → GenericSystem -->
+        <xacro:if value="${sim_backend == 'gazebo'}">
+            <xacro:property name="hw_plugin" value="gazebo_ros2_control/GazeboSystem"/>
+        </xacro:if>
+        <xacro:if value="${sim_backend == 'mock'}">
+            <xacro:property name="hw_plugin" value="mock_components/GenericSystem"/>
+        </xacro:if>
+        <xacro:if value="${sim_backend != 'gazebo' and sim_backend != 'mock'}">
+            <xacro:property name="hw_plugin" value="mock_components/GenericSystem"/>
+        </xacro:if>
         <ros2_control name="${name}" type="system">
             <hardware>
-                <plugin>gazebo_ros2_control/GazeboSystem</plugin>
+                <plugin>${hw_plugin}</plugin>
             </hardware>
             <joint name="J1">
@@ -49,4 +59,18 @@
                 <state_interface name="velocity"/>
             </joint>
+            <joint name="gripper_left_joint">
+                <command_interface name="position"/>
+                <state_interface name="position">
+                  <param name="initial_value">${initial_positions['gripper_left_joint']}</param>
+                </state_interface>
+                <state_interface name="velocity"/>
+            </joint>
+            <joint name="gripper_right_joint">
+                <command_interface name="position"/>
+                <state_interface name="position">
+                  <param name="initial_value">${initial_positions['gripper_right_joint']}</param>
+                </state_interface>
+                <state_interface name="velocity"/>
+            </joint>
         </ros2_control>
     </xacro:macro>

File: src/my_robot_moveit_config/config/episode_urdf_0523.urdf.xacro (robot description, xacro)
@@ -2,8 +2,14 @@
 <robot xmlns:xacro="http://www.ros.org/wiki/xacro" name="episode_urdf_0523">
     <xacro:arg name="initial_positions_file" default="initial_positions.yaml" />
+    <xacro:arg name="sim_backend" default="gazebo" />
     <!-- Import episode_urdf_0523 urdf file -->
     <xacro:include filename="$(find my_robot_moveit_config)/urdf/arm.urdf" />
     <!-- Import control_xacro -->
     <xacro:include filename="episode_urdf_0523.ros2_control.xacro" />
-    <xacro:episode_urdf_0523_ros2_control name="GazeboSystem" initial_positions_file="$(arg initial_positions_file)"/>
+    <!-- Import gripper xacro -->
+    <xacro:include filename="$(find my_robot_moveit_config)/urdf/gripper.xacro" />
+    <xacro:episode_urdf_0523_ros2_control name="GazeboSystem" initial_positions_file="$(arg initial_positions_file)" sim_backend="$(arg sim_backend)"/>
+    <!-- 挂载平行夹爪到 L6 末端，单侧行程 47.5mm → 总开合 95mm -->
+    <xacro:parallel_gripper parent_link="L6" stroke="0.0475"/>
+    <xacro:gripper_transmissions/>
 </robot>

Commit message: 更新夹爪及其机械臂URDF模型、MoveIt配置文件和运动规划代码

File: src/arm_urdf/urdf/arm.urdf (robot description, URDF)
Before this commit: robot episode_urdf_0523, 10 links, 9 joints
Joints:
- joint gripper_right_joint: mimic (none) -> joint=gripper_left_joint multiplier=1 offset=0

File: src/my_robot_moveit_config/config/episode_urdf_0523.ros2_control.xacro (robot description, xacro)
@@ -67,8 +67,12 @@
             </joint>
             <joint name="gripper_right_joint">
-                <command_interface name="position"/>
-                <state_interface name="position">
-                  <param name="initial_value">${initial_positions['gripper_right_joint']}</param>
-                </state_interface>
+                <param name="mimic">gripper_left_joint</param>
+                <param name="multiplier">1.0</param>
+                <command_interface name="position">
+                    <param name="p">1000.0</param>
+                    <param name="i">0.0</param>
+                    <param name="d">10.0</param>
+                </command_interface>
+                <state_interface name="position"/>
                 <state_interface name="velocity"/>
             </joint>

File: src/my_robot_moveit_config/urdf/gripper.xacro (robot description, xacro)
@@ -44,5 +44,5 @@
     </joint>
     <!-- ================================================================ -->
-    <!-- 右手指 — 细长 box，沿 +Y 向中心滑动，独立控制（无 mimic）     -->
+    <!-- 右手指 — 细长 box，沿 +Y 向中心滑动，被动跟随左手指 (mimic) -->
     <!-- ================================================================ -->
     <link name="${prefix}gripper_right">
@@ -68,4 +68,11 @@
       </collision>
     </link>
+  <link name="mimic_dummy_link"/>
+    <joint name="gripper_right_joint_mimic" type="revolute">
+      <parent link="base_link"/>
+      <child link="mimic_dummy_link"/>
+      <axis xyz="0 0 1"/>
+      <limit lower="-3.14" upper="3.14" effort="0" velocity="0"/>
+  </joint>
     <joint name="${prefix}gripper_right_joint" type="prismatic">
       <origin xyz="0.0 -0.05 0.0" rpy="0 0 0"/>
@@ -75,4 +82,5 @@
       <limit lower="0" upper="${stroke}" effort="50" velocity="0.05"/>
       <dynamics damping="2.0" friction="1.0"/>
+      <mimic joint="${prefix}gripper_left_joint" multiplier="1" offset="0"/>
     </joint>
   </xacro:macro>
@@ -88,14 +96,4 @@
       </actuator>
     </transmission>
-    <transmission name="${prefix}trans_gripper_right">
-      <type>transmission_interface/SimpleTransmission</type>
-      <joint name="${prefix}gripper_right_joint">
-        <hardwareInterface>hardware_interface/PositionJointInterface</hardwareInterface>
-      </joint>
-      <actuator name="${prefix}motor_gripper_right">
-        <hardwareInterface>hardware_interface/PositionJointInterface</hardwareInterface>
-        <mechanicalReduction>1</mechanicalReduction>
-      </actuator>
-    </transmission>
   </xacro:macro>
 </robot>
